File: Esquematico V2/Esp_32.sch (KiCad schematic (older format))
At the start: 7 parts

Commit message: Add files via upload
Connections:
- net labels added: 1PPS, RESETGPS, RXD1GPS, TXD1GPS
- wire segments 26 -> 29
Other:
- moved on the sheet: D?, R?
Changed lines of the file:
@@
 L Device:LED D?
 U 1 1 61A9D6F8
-P 5900 3550
+P 7700 3550
 AR Path="/61A89954/61A9D6F8" Ref="D?"  Part="1"
 AR Path="/61A89555/61A9D6F8" Ref="D?"  Part="1"
-F 0 "D?" H 5893 3767 50  0000 C CNN
-F 1 "LED" H 5893 3676 50  0000 C CNN
-F 2 "" H 5900 3550 50  0001 C CNN
-F 3 "~" H 5900 3550 50  0001 C CNN
-	1    5900 3550
+F 0 "D?" H 7693 3767 50  0000 C CNN
+F 1 "LED" H 7693 3676 50  0000 C CNN
+F 2 "" H 7700 3550 50  0001 C CNN
+F 3 "~" H 7700 3550 50  0001 C CNN
+	1    7700 3550
 	-1   0    0    1
 $EndComp
-Wire Wire Line
-	5600 3550 5750 3550
 $Comp
 L power:GND #PWR?
 U 1 1 61AAECDD
-P 6750 3650
-F 0 "#PWR?" H 6750 3400 50  0001 C CNN
-F 1 "GND" H 6755 3477 50  0000 C CNN
-F 2 "" H 6750 3650 50  0001 C CNN
-F 3 "" H 6750 3650 50  0001 C CNN
-	1    6750 3650
+P 8550 3650
+F 0 "#PWR?" H 8550 3400 50  0001 C CNN
+F 1 "GND" H 8555 3477 50  0000 C CNN
+F 2 "" H 8550 3650 50  0001 C CNN
+F 3 "" H 8550 3650 50  0001 C CNN
+	1    8550 3650
 	1    0    0    -1
 $EndComp
 Wire Wire Line
-	6750 3550 6750 3650
-Connection ~ 5750 3550
-Wire Wire Line
-	5750 3550 5850 3550
+	8550 3550 8550 3650
 $Comp
 L Device:R R?
 U 1 1 61AB1DDA
-P 6400 3550
-F 0 "R?" V 6193 3550 50  0000 C CNN
-F 1 "R" V 6284 3550 50  0000 C CNN
-F 2 "" V 6330 3550 50  0001 C CNN
-F 3 "~" H 6400 3550 50  0001 C CNN
-	1    6400 3550
+P 8200 3550
+F 0 "R?" V 7993 3550 50  0000 C CNN
+F 1 "R" V 8084 3550 50  0000 C CNN
+F 2 "" V 8130 3550 50  0001 C CNN
+F 3 "~" H 8200 3550 50  0001 C CNN
+	1    8200 3550
 	0    1    1    0
 $EndComp
 Wire Wire Line
-	6250 3550 6050 3550
+	8050 3550 7850 3550
 Wire Wire Line
-	6550 3550 6750 3550
+	8350 3550 8550 3550
 $Comp
 L Switch:SW_Push_Dual_x2 SW?
@@
 Wire Wire Line
 	5600 3450 6500 3450
+Wire Wire Line
+	5600 3550 7550 3550
+Text HLabel 5850 3650 2    50   Input ~ 0
+1PPS
+Text HLabel 5850 3750 2    50   Input ~ 0
+RXD1GPS
+Text HLabel 5850 3850 2    50   Input ~ 0
+TXD1GPS
+Text HLabel 5850 3950 2    50   Input ~ 0
+RESETGPS
+Wire Wire Line
+	5600 3650 5850 3650
+Wire Wire Line
+	5600 3750 5850 3750
+Wire Wire Line
+	5600 3850 5850 3850
+Wire Wire Line
+	5600 3950 5850 3950
 $EndSCHEMATC
