File: Esquematico V2/Telemetria_apicola.sch (KiCad schematic (older format))
At the start: 0 parts

Commit message: Add files via upload
Changed lines of the file:
@@
 F10 "Microbomba" I L 5400 3000 50
 F11 "Enable_Ventilador_Microbomba" I L 5400 3100 50
+F12 "1PPS" I R 6650 3300 50
+F13 "RXD1GPS" I R 6650 3400 50
+F14 "TXD1GPS" I R 6650 3500 50
+F15 "RESETGPS" I R 6650 3600 50
 $EndSheet
 $Sheet
@@
 	5050 3750 5050 3100
 $Sheet
-S 7000 3700 1150 450
+S 7000 3600 850  550
 U 61B777C0
 F0 "GPS" 50
 F1 "GPS.sch" 50
+F2 "1PPS" I L 7000 3650 50
+F3 "RESETGPS" I L 7000 3750 50
+F4 "RXD1GPS" I L 7000 3850 50
+F5 "TXD1GPS" I L 7000 3950 50
+F6 "CIRCUITODCARGA" I L 7000 4050 50
 $EndSheet
+Wire Wire Line
+	6650 3300 6900 3300
+Wire Wire Line
+	6900 3300 6900 3650
+Wire Wire Line
+	6900 3650 7000 3650
+Wire Wire Line
+	6650 3400 6850 3400
+Wire Wire Line
+	6850 3400 6850 3750
+Wire Wire Line
+	6850 3750 7000 3750
+Wire Wire Line
+	6650 3500 6800 3500
+Wire Wire Line
+	6800 3500 6800 3850
+Wire Wire Line
+	6800 3850 7000 3850
+Wire Wire Line
+	6650 3600 6750 3600
+Wire Wire Line
+	6750 3600 6750 3950
+Wire Wire Line
+	6750 3950 7000 3950
 $EndSCHEMATC
