File: Esquematico/Actuadores.sch (KiCad schematic (older format))
At the start: 2 parts

Commit message: Add files via upload
Parts:
- added J?: Conn_ReleBombilla, symbol Connector:Conn_01x02_Female
Connections:
- net Enable_Ventilador_Microbomba: now also U?.9 (EN3,4)
- net GND: now also J?.2 (Pin_2)
- net ReleBombilla: now reaches U?.10 (3A)
- net at U?.11 (3Y): now also J?.1 (Pin_1)
Changed lines of the file:
@@
 Wire Wire Line
 	6700 2800 7050 2800
+Text HLabel 5150 3750 0    50   Input ~ 0
+Enable_Ventilador_Microbomba
+Wire Wire Line
+	5150 3750 5250 3750
+Text HLabel 5150 3350 0    50   Input ~ 0
+ReleBombilla
+Wire Wire Line
+	5150 3350 5250 3350
+$Comp
+L Connector:Conn_01x02_Female J?
+U 1 1 61B21B3E
+P 7100 3350
+F 0 "J?" H 7128 3326 50  0000 L CNN
+F 1 "Conn_ReleBombilla" H 7128 3235 50  0000 L CNN
+F 2 "" H 7100 3350 50  0001 C CNN
+F 3 "~" H 7100 3350 50  0001 C CNN
+	1    7100 3350
+	1    0    0    -1
+$EndComp
+Wire Wire Line
+	6250 3350 6900 3350
+$Comp
+L power:GND #PWR?
+U 1 1 61B229AF
+P 6900 3550
+F 0 "#PWR?" H 6900 3300 50  0001 C CNN
+F 1 "GND" H 6905 3377 50  0000 C CNN
+F 2 "" H 6900 3550 50  0001 C CNN
+F 3 "" H 6900 3550 50  0001 C CNN
+	1    6900 3550
+	1    0    0    -1
+$EndComp
+Wire Wire Line
+	6900 3450 6900 3550
 $EndSCHEMATC

Commit message: Foot prints
Parts:
- gave numbers to parts that had none: 3
Changed lines of the file:
@@
 $EndDescr
 $Comp
-L Driver_Motor:L293D U?
+L Driver_Motor:L293D U4
 U 1 1 61B6A3A7
 P 5750 3350
-F 0 "U?" H 5750 4531 50  0000 C CNN
+F 0 "U4" H 5750 4531 50  0000 C CNN
 F 1 "L293D" H 5750 4440 50  0000 C CNN
 F 2 "Package_DIP:DIP-16_W7.62mm" H 6000 2600 50  0001 L CNN
@@
 	5650 2050 5850 2050
 $Comp
-L power:GND #PWR?
+L power:GND #PWR0116
 U 1 1 61B6D739
 P 5750 4300
-F 0 "#PWR?" H 5750 4050 50  0001 C CNN
+F 0 "#PWR0116" H 5750 4050 50  0001 C CNN
 F 1 "GND" H 5755 4127 50  0000 C CNN
 F 2 "" H 5750 4300 50  0001 C CNN
@@
 	5150 3150 5250 3150
 $Comp
-L Connector:Conn_01x04_Female J?
+L Connector:Conn_01x04_Female J6
 U 1 1 61B710AD
 P 7250 2700
-F 0 "J?" H 7278 2676 50  0000 L CNN
+F 0 "J6" H 7278 2676 50  0000 L CNN
 F 1 "Conn_Ventilador_Microbomba" H 7278 2585 50  0000 L CNN
 F 2 "" H 7250 2700 50  0001 C CNN
@@
 $EndComp
 $Comp
-L power:GND #PWR?
+L power:GND #PWR0117
 U 1 1 61B71897
 P 6950 3000
-F 0 "#PWR?" H 6950 2750 50  0001 C CNN
+F 0 "#PWR0117" H 6950 2750 50  0001 C CNN
 F 1 "GND" H 6955 2827 50  0000 C CNN
 F 2 "" H 6950 3000 50  0001 C CNN
@@
 	5150 3350 5250 3350
 $Comp
-L Connector:Conn_01x02_Female J?
+L Connector:Conn_01x02_Female J5
 U 1 1 61B21B3E
 P 7100 3350
-F 0 "J?" H 7128 3326 50  0000 L CNN
+F 0 "J5" H 7128 3326 50  0000 L CNN
 F 1 "Conn_ReleBombilla" H 7128 3235 50  0000 L CNN
 F 2 "" H 7100 3350 50  0001 C CNN
@@
 	6250 3350 6900 3350
 $Comp
-L power:GND #PWR?
+L power:GND #PWR0118
 U 1 1 61B229AF
 P 6900 3550
-F 0 "#PWR?" H 6900 3300 50  0001 C CNN
+F 0 "#PWR0118" H 6900 3300 50  0001 C CNN
 F 1 "GND" H 6905 3377 50  0000 C CNN
 F 2 "" H 6900 3550 50  0001 C CNN
