File: Esquematico/Actuadores.sch (KiCad schematic (older format))
At the start: 3 parts, among them J5 Conn_ReleBombilla, J6 Conn_Ventilador_Microbomba, U4 L293D

Commit message: Carga elementos PCB
Parts:
- J5: footprint (none) -> Connector_PinSocket_2.54mm:PinSocket_1x02_P2.54mm_Vertical
- J6: footprint (none) -> Connector_PinSocket_2.54mm:PinSocket_1x04_P2.54mm_Vertical
Changed lines of the file:
@@
 F 0 "J6" H 7278 2676 50  0000 L CNN
 F 1 "Conn_Ventilador_Microbomba" H 7278 2585 50  0000 L CNN
-F 2 "" H 7250 2700 50  0001 C CNN
+F 2 "Connector_PinSocket_2.54mm:PinSocket_1x04_P2.54mm_Vertical" H 7250 2700 50  0001 C CNN
 F 3 "~" H 7250 2700 50  0001 C CNN
 	1    7250 2700
@@
 F 0 "J5" H 7128 3326 50  0000 L CNN
 F 1 "Conn_ReleBombilla" H 7128 3235 50  0000 L CNN
-F 2 "" H 7100 3350 50  0001 C CNN
+F 2 "Connector_PinSocket_2.54mm:PinSocket_1x02_P2.54mm_Vertical" H 7100 3350 50  0001 C CNN
 F 3 "~" H 7100 3350 50  0001 C CNN
 	1    7100 3350
