File: Esquematico/Pantalla.sch (KiCad schematic (older format))
At the start: 1 part

Commit message: Foot prints
Parts:
- J2: renamed from J?; footprint (none) -> Connector_Stocko:Stocko_MKS_1654-6-0-404_1x4_P2.50mm_Vertical
Changed lines of the file:
@@
 P 6100 3700
 AR Path="/61A8D8B4" Ref="J?"  Part="1"
-AR Path="/61A89771/61A8D8B4" Ref="J?"  Part="1"
-F 0 "J?" H 6072 3582 50  0000 R CNN
+AR Path="/61A89771/61A8D8B4" Ref="J2"  Part="1"
+F 0 "J2" H 6072 3582 50  0000 R CNN
 F 1 "Conn_PANTALLA" H 6072 3673 50  0000 R CNN
-F 2 "" H 6100 3700 50  0001 C CNN
+F 2 "Connector_Stocko:Stocko_MKS_1654-6-0-404_1x4_P2.50mm_Vertical" H 6100 3700 50  0001 C CNN
 F 3 "~" H 6100 3700 50  0001 C CNN
 	1    6100 3700
@@
 P 5750 4000
 AR Path="/61A8D8BA" Ref="#PWR?"  Part="1"
-AR Path="/61A89771/61A8D8BA" Ref="#PWR?"  Part="1"
-F 0 "#PWR?" H 5750 3750 50  0001 C CNN
+AR Path="/61A89771/61A8D8BA" Ref="#PWR0102"  Part="1"
+F 0 "#PWR0102" H 5750 3750 50  0001 C CNN
 F 1 "GND" H 5755 3827 50  0000 C CNN
 F 2 "" H 5750 4000 50  0001 C CNN
