File: Esquematico/Reguladores.sch (KiCad schematic (older format))
At the start: 7 parts

Commit message: Foot prints
Parts:
- C3, C4, C5, C6: renamed from C?; footprint (none) -> Capacitor_SMD:C_0805_2012Metric_Pad1.18x1.45mm_HandSolder
- gave numbers to parts that had none: 3
Changed lines of the file:
@@
 $EndDescr
 $Comp
-L Regulator_Linear:AMS1117-3.3 U?
+L Regulator_Linear:AMS1117-3.3 U2
 U 1 1 61B5A9B1
 P 6050 2800
-F 0 "U?" H 6050 3042 50  0000 C CNN
+F 0 "U2" H 6050 3042 50  0000 C CNN
 F 1 "AMS1117-3.3" H 6050 2951 50  0000 C CNN
 F 2 "Package_TO_SOT_SMD:SOT-223-3_TabPin2" H 6050 3000 50  0001 C CNN
@@
 $EndComp
 $Comp
-L Connector:Conn_01x02_Female J?
+L Connector:Conn_01x02_Female J4
 U 1 1 61B5CBA7
 P 5050 2800
-F 0 "J?" H 4942 2985 50  0000 C CNN
+F 0 "J4" H 4942 2985 50  0000 C CNN
 F 1 "Conn_01x02_Female" H 4942 2894 50  0000 C CNN
 F 2 "" H 5050 2800 50  0001 C CNN
@@
 	5250 2800 5650 2800
 $Comp
-L power:GND #PWR?
+L power:GND #PWR0109
 U 1 1 61B5D522
 P 5250 2950
-F 0 "#PWR?" H 5250 2700 50  0001 C CNN
+F 0 "#PWR0109" H 5250 2700 50  0001 C CNN
 F 1 "GND" H 5255 2777 50  0000 C CNN
 F 2 "" H 5250 2950 50  0001 C CNN
@@
 $EndComp
 $Comp
-L power:GND #PWR?
+L power:GND #PWR0110
 U 1 1 61B5DB7A
 P 6050 3150
-F 0 "#PWR?" H 6050 2900 50  0001 C CNN
+F 0 "#PWR0110" H 6050 2900 50  0001 C CNN
 F 1 "GND" H 6055 2977 50  0000 C CNN
 F 2 "" H 6050 3150 50  0001 C CNN
@@
 	5250 2900 5250 2950
 $Comp
-L Device:C C?
+L Device:C C3
 U 1 1 61B5DF8A
 P 6500 3000
-F 0 "C?" H 6615 3046 50  0000 L CNN
+F 0 "C3" H 6615 3046 50  0000 L CNN
 F 1 "10uF" H 6615 2955 50  0000 L CNN
-F 2 "" H 6538 2850 50  0001 C CNN
+F 2 "Capacitor_SMD:C_0805_2012Metric_Pad1.18x1.45mm_HandSolder" H 6538 2850 50  0001 C CNN
 F 3 "~" H 6500 3000 50  0001 C CNN
 	1    6500 3000
@@
 $EndComp
 $Comp
-L Device:C C?
+L Device:C C5
 U 1 1 61B5E49A
 P 6900 3000
-F 0 "C?" H 7015 3046 50  0000 L CNN
+F 0 "C5" H 7015 3046 50  0000 L CNN
 F 1 "0.1uF" H 7015 2955 50  0000 L CNN
-F 2 "" H 6938 2850 50  0001 C CNN
+F 2 "Capacitor_SMD:C_0805_2012Metric_Pad1.18x1.45mm_HandSolder" H 6938 2850 50  0001 C CNN
 F 3 "~" H 6900 3000 50  0001 C CNN
 	1    6900 3000
@@
 Connection ~ 6900 2800
 $Comp
-L power:GND #PWR?
+L power:GND #PWR0111
 U 1 1 61B5ED20
 P 6500 3200
-F 0 "#PWR?" H 6500 2950 50  0001 C CNN
+F 0 "#PWR0111" H 6500 2950 50  0001 C CNN
 F 1 "GND" H 6505 3027 50  0000 C CNN
 F 2 "" H 6500 3200 50  0001 C CNN
@@
 $EndComp
 $Comp
-L power:GND #PWR?
+L power:GND #PWR0112
 U 1 1 61B5F25D
 P 6900 3200
-F 0 "#PWR?" H 6900 2950 50  0001 C CNN
+F 0 "#PWR0112" H 6900 2950 50  0001 C CNN
 F 1 "GND" H 6905 3027 50  0000 C CNN
 F 2 "" H 6900 3200 50  0001 C CNN
@@
 	6500 3150 6500 3200
 $Comp
-L power:GND #PWR?
+L power:GND #PWR0113
 U 1 1 61B65208
 P 6050 4100
-F 0 "#PWR?" H 6050 3850 50  0001 C CNN
+F 0 "#PWR0113" H 6050 3850 50  0001 C CNN
 F 1 "GND" H 6055 3927 50  0000 C CNN
 F 2 "" H 6050 4100 50  0001 C CNN
@@
 	6050 4050 6050 4100
 $Comp
-L Device:C C?
+L Device:C C4
 U 1 1 61B65210
 P 6500 3950
-F 0 "C?" H 6615 3996 50  0000 L CNN
+F 0 "C4" H 6615 3996 50  0000 L CNN
 F 1 "10uF" H 6615 3905 50  0000 L CNN
-F 2 "" H 6538 3800 50  0001 C CNN
+F 2 "Capacitor_SMD:C_0805_2012Metric_Pad1.18x1.45mm_HandSolder" H 6538 3800 50  0001 C CNN
 F 3 "~" H 6500 3950 50  0001 C CNN
 	1    6500 3950
@@
 $EndComp
 $Comp
-L Device:C C?
+L Device:C C6
 U 1 1 61B65216
 P 6900 3950
-F 0 "C?" H 7015 3996 50  0000 L CNN
+F 0 "C6" H 7015 3996 50  0000 L CNN
 F 1 "0.1uF" H 7015 3905 50  0000 L CNN
-F 2 "" H 6938 3800 50  0001 C CNN
+F 2 "Capacitor_SMD:C_0805_2012Metric_Pad1.18x1.45mm_HandSolder" H 6938 3800 50  0001 C CNN
 F 3 "~" H 6900 3950 50  0001 C CNN
 	1    6900 3950
@@
 Connection ~ 6900 3750
 $Comp
-L power:GND #PWR?
+L power:GND #PWR0114
 U 1 1 61B65224
 P 6500 4150
-F 0 "#PWR?" H 6500 3900 50  0001 C CNN
+F 0 "#PWR0114" H 6500 3900 50  0001 C CNN
 F 1 "GND" H 6505 3977 50  0000 C CNN
 F 2 "" H 6500 4150 50  0001 C CNN
@@
 $EndComp
 $Comp
-L power:GND #PWR?
+L power:GND #PWR0115
 U 1 1 61B6522A
 P 6900 4150
-F 0 "#PWR?" H 6900 3900 50  0001 C CNN
+F 0 "#PWR0115" H 6900 3900 50  0001 C CNN
 F 1 "GND" H 6905 3977 50  0000 C CNN
 F 2 "" H 6900 4150 50  0001 C CNN
@@
 	6500 4100 6500 4150
 $Comp
-L Regulator_Linear:AMS1117-5.0 U?
+L Regulator_Linear:AMS1117-5.0 U3
 U 1 1 61B65CA8
 P 6050 3750
-F 0 "U?" H 6050 3992 50  0000 C CNN
+F 0 "U3" H 6050 3992 50  0000 C CNN
 F 1 "AMS1117-5.0" H 6050 3901 50  0000 C CNN
 F 2 "Package_TO_SOT_SMD:SOT-223-3_TabPin2" H 6050 3950 50  0001 C CNN
