File: Esquematico/Sensor_DHT11.sch (KiCad schematic (older format))
At the start: 3 parts

Commit message: Foot prints
Parts:
- C2: renamed from C?; footprint (none) -> Capacitor_SMD:C_0805_2012Metric_Pad1.18x1.45mm_HandSolder
- R3: renamed from R?; footprint (none) -> Resistor_SMD:R_0805_2012Metric_Pad1.20x1.40mm_HandSolder
- gave numbers to parts that had none: 1
Changed lines of the file:
@@
 $EndDescr
 $Comp
-L Connector:Conn_01x04_Female J?
+L Connector:Conn_01x04_Female J3
 U 1 1 61B548CE
 P 6500 3700
-F 0 "J?" H 6528 3676 50  0000 L CNN
+F 0 "J3" H 6528 3676 50  0000 L CNN
 F 1 "Conn_DHT11" H 6528 3585 50  0000 L CNN
 F 2 "" H 6500 3700 50  0001 C CNN
@@
 $EndComp
 $Comp
-L power:GND #PWR?
+L power:GND #PWR0107
 U 1 1 61B55C2A
 P 6300 4000
-F 0 "#PWR?" H 6300 3750 50  0001 C CNN
+F 0 "#PWR0107" H 6300 3750 50  0001 C CNN
 F 1 "GND" H 6305 3827 50  0000 C CNN
 F 2 "" H 6300 4000 50  0001 C CNN
@@
 	6300 3900 6300 4000
 $Comp
-L Device:C C?
+L Device:C C2
 U 1 1 61B56237
 P 5500 3600
-F 0 "C?" V 5248 3600 50  0000 C CNN
+F 0 "C2" V 5248 3600 50  0000 C CNN
 F 1 "100nF" V 5339 3600 50  0000 C CNN
-F 2 "" H 5538 3450 50  0001 C CNN
+F 2 "Capacitor_SMD:C_0805_2012Metric_Pad1.18x1.45mm_HandSolder" H 5538 3450 50  0001 C CNN
 F 3 "~" H 5500 3600 50  0001 C CNN
 	1    5500 3600
@@
 $EndComp
 $Comp
-L power:GND #PWR?
+L power:GND #PWR0108
 U 1 1 61B56D7B
 P 5250 3600
-F 0 "#PWR?" H 5250 3350 50  0001 C CNN
+F 0 "#PWR0108" H 5250 3350 50  0001 C CNN
 F 1 "GND" V 5255 3472 50  0000 R CNN
 F 2 "" H 5250 3600 50  0001 C CNN
@@
 	5650 3600 5700 3600
 $Comp
-L Device:R_Small_US R?
+L Device:R_Small_US R3
 U 1 1 61B574A2
 P 5800 3700
-F 0 "R?" V 5595 3700 50  0000 C CNN
+F 0 "R3" V 5595 3700 50  0000 C CNN
 F 1 "5K" V 5686 3700 50  0000 C CNN
-F 2 "" H 5800 3700 50  0001 C CNN
+F 2 "Resistor_SMD:R_0805_2012Metric_Pad1.20x1.40mm_HandSolder" H 5800 3700 50  0001 C CNN
 F 3 "~" H 5800 3700 50  0001 C CNN
 	1    5800 3700

Commit message: Carga elementos PCB
Parts:
- J3: footprint (none) -> Connector_PinSocket_2.54mm:PinSocket_1x04_P2.54mm_Vertical
Changed lines of the file:
@@
 F 0 "J3" H 6528 3676 50  0000 L CNN
 F 1 "Conn_DHT11" H 6528 3585 50  0000 L CNN
-F 2 "" H 6500 3700 50  0001 C CNN
+F 2 "Connector_PinSocket_2.54mm:PinSocket_1x04_P2.54mm_Vertical" H 6500 3700 50  0001 C CNN
 F 3 "~" H 6500 3700 50  0001 C CNN
 	1    6500 3700
