File: Esquematico/Telemetria_apicola.kicad_pcb (KiCad board)
At the start: 2 copper layers, 50 parts, among them IC1 BQ24070RHLR, J1 Conn_USB, J10 Conn_01x02_Female, J2 Conn_PANTALLA, J3 Conn_DHT11, J5 Conn_ReleBombilla, J6 Conn_Ventilador_Microbomba, J7 Conn_GPS, J8 Conn_01x02_Male, J9 Barrel_Jack_Switch, SW1 SW_EN, SW2 SW_BOOT OPTION, U1 ESP32-WROOM-32, U4 L293D, U5 MT3608, U6 AMS1117-3.3

Commit message: Actualización PCB
Parts:
- added H1: MountingHole, MountingHole:MountingHole_3.2mm_M3_ISO7380, F.Cu at (71.6, 142.2)
- added H2: MountingHole, MountingHole:MountingHole_3.2mm_M3_ISO7380, F.Cu at (170.2, 142.2)
- added H3: MountingHole, MountingHole:MountingHole_3.2mm_M3_ISO7380, F.Cu at (169.7, 76.7)
- added H4: MountingHole, MountingHole:MountingHole_3.2mm_M3_ISO7380, F.Cu at (72.1, 76.7)
- moved J9 5.36 mm to (87.4, 118.9), turned to 270 degrees
Routing:
- net GND: track 476.6 -> 438.3 mm, vias 1 -> 4
- net /CargadorBateria/12V: track 162.0 -> 148.4 mm, vias 2 -> 3
- net Net-(J5-Pad1): track 11.2 -> 14.8 mm, vias 0 -> 2
- net Net-(D5-Pad2): track 134.5 -> 137.9 mm
- net /Esp_32/Sda: track 66.9 -> 64.1 mm, vias 0 -> 1
- net /CargadorBateria/3V3: track 254.5 -> 255.7 mm, vias 1 -> 3
- net Net-(D1-Pad2): track 52.5 -> 53.6 mm, vias 0 -> 1
- net /Actuadores/5V: track 204.4 -> 205.4 mm, vias 1 -> 2
- net Net-(J6-Pad1): track 18.4 -> 18.8 mm, vias 0 -> 2
- net Net-(D1-Pad1): track 9.24 -> 8.93 mm, vias 0 -> 1
- net /Esp_32/Scl: track 64.1 -> 64.3 mm, vias 0 -> 1
- net /CargadorBateria/BAT: track 50.3 -> 50.4 mm, vias 2 -> 3
- net /Esp_32/Tx: vias 2 -> 3
- net /Esp_32/Rx: vias 2 -> 3
- added copper zone on B.Cu, net GND
- added copper zone on F.Cu, net GND
Other:
- board outline added: 107.7 x 76.7 mm

Commit message: Modificacion PCB
Connections:
- U1 pad 23: /Esp_32/RXD1GPS -> Net-(U1-Pad23)
- U1 pad 27: /Esp_32/TXD1GPS -> /Esp_32/RXD1GPS
- U1 pad 28: Net-(U1-Pad28) -> /Esp_32/TXD1GPS
Routing:
- net /Esp_32/RXD1GPS: track 85.4 -> 78.3 mm, vias 1 -> 3
- net GND: track 438.3 -> 435.7 mm, vias 4 -> 5
- net /Actuadores/Microbomba: track 33.1 -> 33.9 mm
- net /Actuadores/5V: track 205.4 -> 206.0 mm
- net /Esp_32/TXD1GPS: track 80.0 -> 79.5 mm
